Commit message: forgot

File: hector_quadrotor_description/urdf/quadrotor_with_asus_with_hokuyo_utm30lx.urdf.xacro (robot description, xacro)
@@ -14,5 +14,11 @@
     <xacro:include filename="$(find hector_sensors_description)/urdf/asus_camera.urdf.xacro" />
     <xacro:asus_camera name="camera" parent="base_link">
-      <origin xyz="0.1 0.0 -0.03" rpy="0 ${M_PI/9} 0"/>
+      <origin xyz="0.1 0.0 -0.03" rpy="0 ${M_PI/6} 0"/>
     </xacro:asus_camera>
+    <!--
+    <xacro:include filename="$(find hector_sensors_description)/urdf/asus_camera.urdf.xacro" />
+    <xacro:asus_camera name="camera2" parent="base_link">
+      <origin xyz="-0.1 0.0 -0.03" rpy="0 ${M_PI/9} ${M_PI}"/>
+    </xacro:asus_camera>
+    -->
 </robot>
